File: pcb/dc_motor.sch (KiCad schematic (older format))
At the start: 36 parts, among them J1 Conn_01x02, J2 Conn_01x09, J3 Conn_01x02, Q1 Q_PMOS_DGS, Q2 BTN8982TA, Q3 BTN8982TA, U1 74AHC244, U2 L7805, U3 INA226

Commit message: project folder
Parts:
- removed C6: C, symbol Device:C
- removed F1: Fuse, symbol Device:Fuse
- removed J2: Conn_01x09, symbol Connector_Generic:Conn_01x09
- removed J3: Conn_01x02, symbol Connector_Generic:Conn_01x02
- removed Q3: BTN8982TA, Package_TO_SOT_SMD:TO-263-7_TabPin8, symbol Power_Management:BTN8982TA
- removed R13, R14: R, symbol Device:R
- added C? (x11): C, symbol Device:C
- added FID? (x4): Fiducial, symbol Mechanical:Fiducial
- added H? (x4): MountingHole, symbol Mechanical:MountingHole
- added J? (x2): Conn_01x04, symbol Connector_Generic:Conn_01x04
- added J?: Conn_01x07, symbol Connector_Generic:Conn_01x07
- added Q?: BTN8982TA, Package_TO_SOT_SMD:TO-263-7_TabPin8, symbol Power_Management:BTN8982TA
- added R? (x8): R, symbol Device:R
Connections:
- net labels added: VMOTOR
- net labels removed: Vin-
- wire segments 124 -> 177
Other:
- note added: "ADC channel"
- note added: "Inverse polarity protection"
- note added: "Mechanical components"
- note added: "Outputs capacity:\n1 dc motor bi directional between 1-4\n2 dc motor uni directional (1-2) (4-3)\n8-30 V @30A max current (PCB limited)\nPWM 30KHz max"
- note added: "Power Monitor\n"
- note added: "VCC\n8-30v\n30A"
- note removed: "Current Sense\n"
- note removed: "Inverse Polarity"
- note removed: "Protection"
- note removed: "Short Circuit Protection"
- moved on the sheet: C1, C2, C3, C4, C5, C7, D1, D2, D3, D4, J1, JP1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
