File: pcb/dc_motor.sch (KiCad schematic (older format))
At the start: 60 parts, among them J1 Conn_01x02, J2 Conn_01x04, J3 Conn_01x04, J4 Conn_01x07, Q1 Q_PMOS_DGS, Q2 BTN8982TA, Q3 BTN8982TA, U1 L7805, U2 INA226, U3 74AHC244

Commit message: sch values
Parts:
- added C?: C, symbol Device:C
- added JP?: EN option, symbol Device:Jumper_NC_Dual
- C1, C10, C13, C15, C16, C17, C2, C5: value C -> 100nF
- C11, C12, C14, C7, C8, C9: value C -> 220nF
- C4: value C -> 330nF
- C6: value CP -> 1000uF/35V
- D1: value D_Zener -> 10V
- D2: value LED -> Power
- D3: value LED -> RIGTH
- D4: value LED -> LEFT
- R1, R10, R2, R3, R9: value R -> 4k7
- R11, R12, R4: value R -> 3k3
- R13, R14, R15, R16, R7: value R -> 10k
- R17, R18: value R -> 1k
- R19, R20: value R -> 470R
- R5, R8: value R -> 10R
- R6: value R -> 10mR
Connections:
- net EN_1: now also JP?.1
- net EN_2: now also JP?.3; no longer R13.1, U3.8 (1A3)
- net GND: now also C?.2
- net at C3.1, J1.1 (Pin_1), Q1.1 (D): now also C?.1
- new net: JP?.2, R13.1, U3.8 (1A3)
Other:
- note added: "Enable outputs\nInvidual or Paralell\nwith EN_1"
- note added: "OUTPUT DIRECTION"
- note added: "Slew Rate"
- note added: "VCC:\n8-30v\n30A"
- note removed: "OUTPUT ENABLE/DIRECTION"
- note removed: "VCC\n8-30v\n30A"
- moved on the sheet: C1, C15, C3, C6, D3, D4, J1, R10, R11, R12, R13, R14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

Commit message: footprints
Parts:
- removed Q1: Q_PMOS_DGS, symbol Device:Q_PMOS_DGS
- added Q1: Q_PMOS_GDS, Package_TO_SOT_SMD:TO-252-2, symbol Device:Q_PMOS_GDS
- C1, U1: footprint (none) -> Package_TO_SOT_SMD:TO-252-2
- C10: renamed from C15; footprint (none) -> Capacitor_SMD:C_0805_2012Metric
- C11: renamed from C9; footprint (none) -> Capacitor_SMD:C_0805_2012Metric
- C12: renamed from C10; footprint (none) -> Capacitor_SMD:C_0805_2012Metric
- C13: renamed from C11; footprint (none) -> Capacitor_SMD:C_0805_2012Metric
- C14: renamed from C12; footprint (none) -> Capacitor_SMD:C_0805_2012Metric
- C15: renamed from C13; footprint (none) -> Capacitor_SMD:C_0805_2012Metric
- C16: renamed from C14; footprint (none) -> Capacitor_SMD:C_0805_2012Metric
- C17: renamed from C16; footprint (none) -> Capacitor_SMD:C_0805_2012Metric
- C18: renamed from C17; footprint (none) -> Capacitor_SMD:C_0805_2012Metric
- C2: footprint (none) -> Capacitor_SMD:C_0805_2012Metric
- C3: renamed from C?; value C -> 10uF; footprint (none) -> Capacitor_SMD:C_0805_2012Metric
- C4: renamed from C3; value C -> 10uF; footprint (none) -> Capacitor_SMD:C_0805_2012Metric
- C5: renamed from C6; footprint (none) -> Capacitor_THT:CP_Radial_D12.5mm_P7.50mm
- C6: renamed from C4; footprint (none) -> Capacitor_SMD:C_0805_2012Metric
- C7: renamed from C5; footprint (none) -> Capacitor_SMD:C_0805_2012Metric
- C8: renamed from C7; footprint (none) -> Capacitor_SMD:C_0805_2012Metric
- C9: renamed from C8; footprint (none) -> Capacitor_SMD:C_0805_2012Metric
- D1: footprint (none) -> Diode_SMD:D_SOD-323
- D2, D3, D4: footprint (none) -> LED_SMD:LED_0805_2012Metric
- FID1, FID2, FID3, FID4: footprint (none) -> Fiducial:Fiducial_0.5mm_Mask1.5mm
- H1, H2, H3, H4: footprint (none) -> MountingHole:MountingHole_3.2mm_M3_ISO14580
- J1: footprint (none) -> Connector_Phoenix_MSTB:PhoenixContact_MSTBVA_2,5_2-G-5,08_1x02_P5.08mm_Vertical
- J2: footprint (none) -> Connector_Phoenix_MSTB:PhoenixContact_MSTBVA_2,5_4-G-5,08_1x04_P5.08mm_Vertical
- J3: footprint (none) -> Connector_Molex:Molex_KK-254_AE-6410-04A_1x04_P2.54mm_Vertical
- J4: footprint (none) -> Connector_Molex:Molex_KK-254_AE-6410-07A_1x07_P2.54mm_Vertical
- JP1: footprint (none) -> Jumper:SolderJumper-3_P1.3mm_Open_RoundedPad1.0x1.5mm
- JP2: renamed from JP?; footprint (none) -> Jumper:SolderJumper-3_P1.3mm_Bridged2Bar12_RoundedPad1.0x1.5mm
- R1, R10, R11, R12, R13, R14, R15, R16, R17, R18, R19, R2, R20, R3, R4, R5, R7, R8, R9: footprint (none) -> Resistor_SMD:R_0805_2012Metric
- R6: footprint (none) -> Resistor_SMD:R_4020_10251Metric
- U3: footprint (none) -> Package_SO:SSOP-20_4.4x6.5mm_P0.65mm
Connections:
- net GND: now also J2.1 (Pin_1), J2.4 (Pin_4); no longer J2.2 (Pin_2), J2.3 (Pin_3)
- net VCC: now also Q1.3 (S)
- net at C13.1, C8.2, Q2.4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: now also J2.2 (Pin_2); no longer J2.1 (Pin_1)
- net at C3.1, C4.1, J1.1 (Pin_1): now also Q1.2 (D)
- net at D1.2 (A), R7.1: now also Q1.1 (G)
- net at C14.1, C9.2, Q3.4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: now also J2.3 (Pin_3); no longer J2.4 (Pin_4)
- net VMOTOR renamed Vdrive
Other:
- moved on the sheet: D1

Commit message: Sch complete.
first revision.
Parts:
- removed C6: 330nF, Capacitor_SMD:C_0805_2012Metric, symbol Device:C
- removed JP2: EN option, Jumper:SolderJumper-3_P1.3mm_Bridged2Bar12_RoundedPad1.0x1.5mm, symbol Device:Jumper_NC_Dual
- added C3, C4, C5: 100nF, Capacitor_SMD:C_0603_1608Metric, symbol Device:C
- added JP2: EN_Option, Connector_PinHeader_2.54mm:PinHeader_1x03_P2.54mm_Vertical, symbol Jumper:Jumper_3_Open
- C1: footprint Package_TO_SOT_SMD:TO-252-2 -> Capacitor_SMD:C_0603_1608Metric; Manufacturer Part Number (none) -> GMK107B7104KAHT; Supplier 1 Part Number (none) -> 587-3354-1-ND
- C10: renamed from C8; footprint Capacitor_SMD:C_0805_2012Metric -> Capacitor_SMD:C_0603_1608Metric; Manufacturer Part Number (none) -> GCJ188R71H224KA01D; Supplier 1 Part Number (none) -> 490-14410-1-ND
- C11: renamed from C9; footprint Capacitor_SMD:C_0805_2012Metric -> Capacitor_SMD:C_0603_1608Metric; Manufacturer Part Number (none) -> GCJ188R71H224KA01D; Supplier 1 Part Number (none) -> 490-14410-1-ND
- C12: renamed from C10; footprint Capacitor_SMD:C_0805_2012Metric -> Capacitor_SMD:C_0603_1608Metric; Manufacturer Part Number (none) -> GMK107B7104KAHT; Supplier 1 Part Number (none) -> 587-3354-1-ND
- C13: renamed from C11; footprint Capacitor_SMD:C_0805_2012Metric -> Capacitor_SMD:C_0603_1608Metric; Manufacturer Part Number (none) -> GCJ188R71H224KA01D; Supplier 1 Part Number (none) -> 490-14410-1-ND
- C14: renamed from C12; footprint Capacitor_SMD:C_0805_2012Metric -> Capacitor_SMD:C_0603_1608Metric; Manufacturer Part Number (none) -> GMK107B7104KAHT; Supplier 1 Part Number (none) -> 587-3354-1-ND
- C15: renamed from C13; footprint Capacitor_SMD:C_0805_2012Metric -> Capacitor_SMD:C_0603_1608Metric; Manufacturer Part Number (none) -> GCJ188R71H224KA01D; Supplier 1 Part Number (none) -> 490-14410-1-ND
- C16: renamed from C14; footprint Capacitor_SMD:C_0805_2012Metric -> Capacitor_SMD:C_0603_1608Metric; Manufacturer Part Number (none) -> GCJ188R71H224KA01D; Supplier 1 Part Number (none) -> 490-14410-1-ND
- C17: renamed from C15; footprint Capacitor_SMD:C_0805_2012Metric -> Capacitor_SMD:C_0603_1608Metric; Manufacturer Part Number (none) -> GMK107B7104KAHT; Supplier 1 Part Number (none) -> 587-3354-1-ND
- C18: renamed from C16; footprint Capacitor_SMD:C_0805_2012Metric -> Capacitor_SMD:C_0603_1608Metric; Manufacturer Part Number (none) -> GCJ188R71H224KA01D; Supplier 1 Part Number (none) -> 490-14410-1-ND
- C19: renamed from C17; footprint Capacitor_SMD:C_0805_2012Metric -> Capacitor_SMD:C_0603_1608Metric; Manufacturer Part Number (none) -> GMK107B7104KAHT; Supplier 1 Part Number (none) -> 587-3354-1-ND
- C2: footprint Capacitor_SMD:C_0805_2012Metric -> Capacitor_SMD:C_0603_1608Metric; Manufacturer Part Number (none) -> GMK107B7104KAHT; Supplier 1 Part Number (none) -> 587-3354-1-ND
- C20: renamed from C18; footprint Capacitor_SMD:C_0805_2012Metric -> Capacitor_SMD:C_0603_1608Metric; Manufacturer Part Number (none) -> GMK107B7104KAHT; Supplier 1 Part Number (none) -> 587-3354-1-ND
- C6: renamed from C7; footprint Capacitor_SMD:C_0805_2012Metric -> Capacitor_SMD:C_0603_1608Metric; Manufacturer Part Number (none) -> GMK107B7104KAHT; Supplier 1 Part Number (none) -> 587-3354-1-ND
- C7: renamed from C3; Manufacturer Part Number (none) -> GCM21BR71A106KE22L; Supplier 1 Part Number (none) -> 490-10674-1-ND
- C8: renamed from C4; Manufacturer Part Number (none) -> GCM21BR71A106KE22L; Supplier 1 Part Number (none) -> 490-10674-1-ND
- C9: renamed from C5; footprint Capacitor_THT:CP_Radial_D12.5mm_P7.50mm -> Capacitor_THT:CP_Radial_D10.0mm_P5.00mm; Manufacturer Part Number (none) -> 35PX1000MEFC10X20; Supplier 1 Part Number (none) -> 1189-1745-ND
- D1: footprint Diode_SMD:D_SOD-323 -> Diode_SMD:D_SOD-123; Manufacturer Part Number (none) -> SZMMSZ5240BT1G; Supplier 1 Part Number (none) -> SZMMSZ5240BT1GOSCT-ND
- D2: footprint LED_SMD:LED_0805_2012Metric -> LED_SMD:LED_0603_1608Metric; Manufacturer Part Number (none) -> LTST-C191KGKT; Supplier 1 Part Number (none) -> 160-1446-1-ND
- D3: footprint LED_SMD:LED_0805_2012Metric -> LED_SMD:LED_0603_1608Metric; Manufacturer Part Number (none) -> LTST-C191KSKT; Supplier 1 Part Number (none) -> 160-1448-1-ND
- D4: footprint LED_SMD:LED_0805_2012Metric -> LED_SMD:LED_0603_1608Metric; Manufacturer Part Number (none) -> LTST-C194TBKT; Supplier 1 Part Number (none) -> 160-1837-1-ND
- FID1, FID2, FID3, FID4, H1, H2, H3, H4, JP1: Manufacturer Part Number (none) -> NF; Supplier 1 Part Number (none) -> NF
- J1: Manufacturer Part Number (none) -> 1758018; Supplier 1 Part Number (none) -> 277-1128-ND
- J2: Manufacturer Part Number (none) -> OQ0453500000G; Supplier 1 Part Number (none) -> 609-4277-ND
- J3: Manufacturer Part Number (none) -> 0022232041; Supplier 1 Part Number (none) -> WM4202-ND
- J4: Manufacturer Part Number (none) -> 0022053071; Supplier 1 Part Number (none) -> WM4305-ND
- Q1: Manufacturer Part Number (none) -> IPD90P03P4L04ATMA1; Supplier 1 Part Number (none) -> IPD90P03P4L04ATMA1CT-ND
- Q2, Q3: Manufacturer Part Number (none) -> BTN8982TAAUMA1; Supplier 1 Part Number (none) -> BTN8982TAAUMA1INCT-ND
- R1, R10, R2, R3, R9: footprint Resistor_SMD:R_0805_2012Metric -> Resistor_SMD:R_0603_1608Metric; Manufacturer Part Number (none) -> RC0603JR-074K7L; Supplier 1 Part Number (none) -> 311-4.7KGRCT-ND
- R11, R12, R4: footprint Resistor_SMD:R_0805_2012Metric -> Resistor_SMD:R_0603_1608Metric; Manufacturer Part Number (none) -> RC0603JR-073K3L; Supplier 1 Part Number (none) -> 311-3.3KGRCT-ND
- R13, R14, R15, R16, R7: footprint Resistor_SMD:R_0805_2012Metric -> Resistor_SMD:R_0603_1608Metric; Manufacturer Part Number (none) -> RC0603FR-0710KL; Supplier 1 Part Number (none) -> 311-10.0KHRCT-ND
- R17, R18: footprint Resistor_SMD:R_0805_2012Metric -> Resistor_SMD:R_0603_1608Metric; Manufacturer Part Number (none) -> RC0603FR-071KL; Supplier 1 Part Number (none) -> 311-1.00KHRCT-ND
- R19, R20: footprint Resistor_SMD:R_0805_2012Metric -> Resistor_SMD:R_0603_1608Metric; Manufacturer Part Number (none) -> RC0603FR-07470RL; Supplier 1 Part Number (none) -> 311-470HRCT-ND
- R5, R8: footprint Resistor_SMD:R_0805_2012Metric -> Resistor_SMD:R_0603_1608Metric; Manufacturer Part Number (none) -> RC0603FR-0710RL; Supplier 1 Part Number (none) -> 311-10.0HRCT-ND
- R6: footprint Resistor_SMD:R_4020_10251Metric -> Resistor_SMD:R_2512_6332Metric; Manufacturer Part Number (none) -> CRA2512-FZ-R010ELF; Supplier 1 Part Number (none) -> CRA2512-FZ-R010ELFCT-ND
- U1: footprint Package_TO_SOT_SMD:TO-252-2 -> Package_TO_SOT_SMD:TO-252-3_TabPin2; Manufacturer Part Number (none) -> L7805CDT-TR; Supplier 1 Part Number (none) -> 497-7255-1-ND
- U2: Manufacturer Part Number (none) -> INA226AIDGST; Supplier 1 Part Number (none) -> 296-29100-1-ND
- U3: footprint Package_SO:SSOP-20_4.4x6.5mm_P0.65mm -> Package_SO:TSSOP-20_4.4x6.5mm_P0.65mm; Manufacturer Part Number (none) -> SN74AHC244QPWRQ1; Supplier 1 Part Number (none) -> SN74AHC244QPWRQ1CT-ND
Connections:
- net EN_1: now also JP2.1 (A)
- net EN_2: now also JP2.3 (B)
- net GND: now also C3.2, C4.2, C5.2
- net VCC: now also C3.1, C4.1, C5.1
- net at R13.1, U3.8 (1A3): now also JP2.2 (C)
Other:
- moved on the sheet: C6, D2, R4, U1

Commit message: Part number changes
Parts:
- C7, C8: Manufacturer Part Number GCM21BR71A106KE22L -> GMK212BBJ106KG-T; Supplier 1 Part Number 490-10674-1-ND -> 587-4893-1-ND
Changed lines of the file:
@@
 F 2 "Capacitor_SMD:C_0805_2012Metric" H 2088 2150 50  0001 C CNN
 F 3 "~" H 2050 2300 50  0001 C CNN
-F 4 "GCM21BR71A106KE22L" H 2050 2300 50  0001 C CNN "Manufacturer Part Number"
-F 5 "490-10674-1-ND" H 2050 2300 50  0001 C CNN "Supplier 1 Part Number"
+F 4 "GMK212BBJ106KG-T" H 2050 2300 50  0001 C CNN "Manufacturer Part Number"
+F 5 "587-4893-1-ND" H 2050 2300 50  0001 C CNN "Supplier 1 Part Number"
 	1    2050 2300
 	1    0    0    -1
@@
 F 2 "Capacitor_SMD:C_0805_2012Metric" H 1838 2150 50  0001 C CNN
 F 3 "~" H 1800 2300 50  0001 C CNN
-F 4 "GCM21BR71A106KE22L" H 1800 2300 50  0001 C CNN "Manufacturer Part Number"
-F 5 "490-10674-1-ND" H 1800 2300 50  0001 C CNN "Supplier 1 Part Number"
+F 4 "GMK212BBJ106KG-T" H 1800 2300 50  0001 C CNN "Manufacturer Part Number"
+F 5 "587-4893-1-ND" H 1800 2300 50  0001 C CNN "Supplier 1 Part Number"
 	1    1800 2300
 	1    0    0    -1
