File: pcb/dc_motor.sch (KiCad schematic (older format))
At the start: 63 parts, among them J1 Conn_01x02, J2 Conn_01x04, J3 Conn_01x04, J4 Conn_01x07, Q1 IPD90P03P4L04, Q2 BTN8982TA, Q3 BTN8982TA, U1 L7805, U2 INA226, U3 74AHC244

Commit message: interactive component place
Parts:
- FID1, FID2, FID3, FID4, H1, H2, H3, H4, JP1: Manufacturer Part Number NF -> dnp; Supplier 1 Part Number NF -> dnp
- LOGO1: Manufacturer Part Number (none) -> dnp; Supplier 1 Part Number (none) -> dnp
Changed lines of the file:
@@
 F 2 "Jumper:SolderJumper-3_P1.3mm_Open_RoundedPad1.0x1.5mm" H 9000 1750 50  0001 C CNN
 F 3 "" H 9000 1750 50  0001 C CNN
-F 4 "NF" H 9000 1750 50  0001 C CNN "Manufacturer Part Number"
-F 5 "NF" H 9000 1750 50  0001 C CNN "Supplier 1 Part Number"
+F 4 "dnp" H 9000 1750 50  0001 C CNN "Manufacturer Part Number"
+F 5 "dnp" H 9000 1750 50  0001 C CNN "Supplier 1 Part Number"
 	1    9000 1750
 	1    0    0    1
@@
 F 2 "MountingHole:MountingHole_3.2mm_M3_ISO14580" H 2900 7050 50  0001 C CNN
 F 3 "~" H 2900 7050 50  0001 C CNN
-F 4 "NF" H 2900 7050 50  0001 C CNN "Manufacturer Part Number"
-F 5 "NF" H 2900 7050 50  0001 C CNN "Supplier 1 Part Number"
+F 4 "dnp" H 2900 7050 50  0001 C CNN "Manufacturer Part Number"
+F 5 "dnp" H 2900 7050 50  0001 C CNN "Supplier 1 Part Number"
 	1    2900 7050
 	1    0    0    -1
@@
 F 2 "MountingHole:MountingHole_3.2mm_M3_ISO14580" H 3350 7050 50  0001 C CNN
 F 3 "~" H 3350 7050 50  0001 C CNN
-F 4 "NF" H 3350 7050 50  0001 C CNN "Manufacturer Part Number"
-F 5 "NF" H 3350 7050 50  0001 C CNN "Supplier 1 Part Number"
+F 4 "dnp" H 3350 7050 50  0001 C CNN "Manufacturer Part Number"
+F 5 "dnp" H 3350 7050 50  0001 C CNN "Supplier 1 Part Number"
 	1    3350 7050
 	1    0    0    -1
@@
 F 2 "MountingHole:MountingHole_3.2mm_M3_ISO14580" H 3900 7050 50  0001 C CNN
 F 3 "~" H 3900 7050 50  0001 C CNN
-F 4 "NF" H 3900 7050 50  0001 C CNN "Manufacturer Part Number"
-F 5 "NF" H 3900 7050 50  0001 C CNN "Supplier 1 Part Number"
+F 4 "dnp" H 3900 7050 50  0001 C CNN "Manufacturer Part Number"
+F 5 "dnp" H 3900 7050 50  0001 C CNN "Supplier 1 Part Number"
 	1    3900 7050
 	1    0    0    -1
@@
 F 2 "MountingHole:MountingHole_3.2mm_M3_ISO14580" H 4400 7050 50  0001 C CNN
 F 3 "~" H 4400 7050 50  0001 C CNN
-F 4 "NF" H 4400 7050 50  0001 C CNN "Manufacturer Part Number"
-F 5 "NF" H 4400 7050 50  0001 C CNN "Supplier 1 Part Number"
+F 4 "dnp" H 4400 7050 50  0001 C CNN "Manufacturer Part Number"
+F 5 "dnp" H 4400 7050 50  0001 C CNN "Supplier 1 Part Number"
 	1    4400 7050
 	1    0    0    -1
@@
 F 2 "Fiducial:Fiducial_0.5mm_Mask1.5mm" H 2900 6750 50  0001 C CNN
 F 3 "~" H 2900 6750 50  0001 C CNN
-F 4 "NF" H 2900 6750 50  0001 C CNN "Manufacturer Part Number"
-F 5 "NF" H 2900 6750 50  0001 C CNN "Supplier 1 Part Number"
+F 4 "dnp" H 2900 6750 50  0001 C CNN "Manufacturer Part Number"
+F 5 "dnp" H 2900 6750 50  0001 C CNN "Supplier 1 Part Number"
 	1    2900 6750
 	1    0    0    -1
@@
 F 2 "Fiducial:Fiducial_0.5mm_Mask1.5mm" H 3400 6750 50  0001 C CNN
 F 3 "~" H 3400 6750 50  0001 C CNN
-F 4 "NF" H 3400 6750 50  0001 C CNN "Manufacturer Part Number"
-F 5 "NF" H 3400 6750 50  0001 C CNN "Supplier 1 Part Number"
+F 4 "dnp" H 3400 6750 50  0001 C CNN "Manufacturer Part Number"
+F 5 "dnp" H 3400 6750 50  0001 C CNN "Supplier 1 Part Number"
 	1    3400 6750
 	1    0    0    -1
@@
 F 2 "Fiducial:Fiducial_0.5mm_Mask1.5mm" H 3900 6750 50  0001 C CNN
 F 3 "~" H 3900 6750 50  0001 C CNN
-F 4 "NF" H 3900 6750 50  0001 C CNN "Manufacturer Part Number"
-F 5 "NF" H 3900 6750 50  0001 C CNN "Supplier 1 Part Number"
+F 4 "dnp" H 3900 6750 50  0001 C CNN "Manufacturer Part Number"
+F 5 "dnp" H 3900 6750 50  0001 C CNN "Supplier 1 Part Number"
 	1    3900 6750
 	1    0    0    -1
@@
 F 2 "Fiducial:Fiducial_0.5mm_Mask1.5mm" H 4400 6750 50  0001 C CNN
 F 3 "~" H 4400 6750 50  0001 C CNN
-F 4 "NF" H 4400 6750 50  0001 C CNN "Manufacturer Part Number"
-F 5 "NF" H 4400 6750 50  0001 C CNN "Supplier 1 Part Number"
+F 4 "dnp" H 4400 6750 50  0001 C CNN "Manufacturer Part Number"
+F 5 "dnp" H 4400 6750 50  0001 C CNN "Supplier 1 Part Number"
 	1    4400 6750
 	1    0    0    -1
@@
 F 2 "Symbol:OSHW-Logo2_9.8x8mm_SilkScreen" H 2050 6900 50  0001 C CNN
 F 3 "~" H 2050 6900 50  0001 C CNN
+F 4 "dnp" H 2050 6900 50  0001 C CNN "Manufacturer Part Number"
+F 5 "dnp" H 2050 6900 50  0001 C CNN "Supplier 1 Part Number"
 	1    2050 6900
 	1    0    0    -1

Commit message: symbols field
Parts:
- C1, C12, C14, C17, C19, C2, C20, C3, C6: #digikey (none) -> 587-3354-1-ND; Manufacturer Part Number GMK107B7104KAHT -> (none); Supplier 1 Part Number 587-3354-1-ND -> (none); manf# (none) -> GMK107B7104KAHT
- C10, C11, C15, C16: #digikey (none) -> 490-14410-1-ND; Manufacturer Part Number GCJ188R71H224KA01D -> (none); Supplier 1 Part Number 490-14410-1-ND -> (none); manf# (none) -> GCJ188R71H224KA01D
- C13, C18: #digikey (none) -> 490-14360-1-ND; Manufacturer Part Number GCM188R91H102KA37D -> (none); Supplier 1 Part Number 490-14360-1-ND -> (none); manf# (none) -> GCM188R91H102KA37D
- C7, C8: #digikey (none) -> 587-4893-1-ND; Manufacturer Part Number GMK212BBJ106KG-T -> (none); Supplier 1 Part Number 587-4893-1-ND -> (none); manf# (none) -> GMK212BBJ106KG-T
- C9: #digikey (none) -> 1189-1745-ND; Manufacturer Part Number 35PX1000MEFC10X20 -> (none); Supplier 1 Part Number 1189-1745-ND -> (none); manf# (none) -> 35PX1000MEFC10X20
- D1: #digikey (none) -> SZMMSZ5240BT1GOSCT-ND; Manufacturer Part Number SZMMSZ5240BT1G -> (none); Supplier 1 Part Number SZMMSZ5240BT1GOSCT-ND -> (none); manf# (none) -> SZMMSZ5240BT1G
- D2: #digikey (none) -> 160-1446-1-ND; Manufacturer Part Number LTST-C191KGKT -> (none); Supplier 1 Part Number 160-1446-1-ND -> (none); manf# (none) -> LTST-C191KGKT
- D3: #digikey (none) -> 160-1448-1-ND; Manufacturer Part Number LTST-C191KSKT -> (none); Supplier 1 Part Number 160-1448-1-ND -> (none); manf# (none) -> LTST-C191KSKT
- D4: #digikey (none) -> 160-1837-1-ND; Manufacturer Part Number LTST-C194TBKT -> (none); Supplier 1 Part Number 160-1837-1-ND -> (none); manf# (none) -> LTST-C194TBKT
- FID1, FID2, FID3, FID4, H1, H2, H3, H4, JP1, LOGO1: #digikey (none) -> dnp; Manufacturer Part Number dnp -> (none); Supplier 1 Part Number dnp -> (none); manf# (none) -> dnp
- J1: #digikey (none) -> 277-1128-ND; Manufacturer Part Number 1758018 -> (none); Supplier 1 Part Number 277-1128-ND -> (none); manf# (none) -> 1758018
- J2: #digikey (none) -> 609-4277-ND; Manufacturer Part Number OQ0453500000G -> (none); Supplier 1 Part Number 609-4277-ND -> (none); manf# (none) -> OQ0453500000G
- J3: #digikey (none) -> WM4202-ND; Manufacturer Part Number 0022232041 -> (none); Supplier 1 Part Number WM4202-ND -> (none); manf# (none) -> 0022232041
- J4: #digikey (none) -> WM4305-ND; Manufacturer Part Number 0022053071 -> (none); Supplier 1 Part Number WM4305-ND -> (none); manf# (none) -> 0022053071
- JP2: #digikey (none) -> 732-5316-ND; Manufacturer Part Number 61300311121 -> (none); Supplier 1 Part Number 732-5316-ND -> (none); manf# (none) -> 61300311121
- Q1: #digikey (none) -> IPD90P03P4L04ATMA1CT-ND; Manufacturer Part Number IPD90P03P4L04ATMA1 -> (none); Supplier 1 Part Number IPD90P03P4L04ATMA1CT-ND -> (none); manf# (none) -> IPD90P03P4L04ATMA1
- Q2, Q3: #digikey (none) -> BTN8982TAAUMA1INCT-ND; Manufacturer Part Number BTN8982TAAUMA1 -> (none); Supplier 1 Part Number BTN8982TAAUMA1INCT-ND -> (none); manf# (none) -> BTN8982TAAUMA1
- R1, R10, R2, R3, R9: #digikey (none) -> 311-4.7KGRCT-ND; Manufacturer Part Number RC0603JR-074K7L -> (none); Supplier 1 Part Number 311-4.7KGRCT-ND -> (none); manf# (none) -> RC0603JR-074K7L
- R11, R12, R4: #digikey (none) -> 311-3.3KGRCT-ND; Manufacturer Part Number RC0603JR-073K3L -> (none); Supplier 1 Part Number 311-3.3KGRCT-ND -> (none); manf# (none) -> RC0603JR-073K3L
- R13, R14, R15, R16, R7: #digikey (none) -> 311-10.0KHRCT-ND; Manufacturer Part Number RC0603FR-0710KL -> (none); Supplier 1 Part Number 311-10.0KHRCT-ND -> (none); manf# (none) -> RC0603FR-0710KL
- R17, R18: #digikey (none) -> 311-1.00KHRCT-ND; Manufacturer Part Number RC0603FR-071KL -> (none); Supplier 1 Part Number 311-1.00KHRCT-ND -> (none); manf# (none) -> RC0603FR-071KL
- R19, R20: #digikey (none) -> 311-470HRCT-ND; Manufacturer Part Number RC0603FR-07470RL -> (none); Supplier 1 Part Number 311-470HRCT-ND -> (none); manf# (none) -> RC0603FR-07470RL
- R5, R8: #digikey (none) -> 311-10.0HRCT-ND; Manufacturer Part Number RC0603FR-0710RL -> (none); Supplier 1 Part Number 311-10.0HRCT-ND -> (none); manf# (none) -> RC0603FR-0710RL
- R6: #digikey (none) -> CRA2512-FZ-R010ELFCT-ND; Manufacturer Part Number CRA2512-FZ-R010ELF -> (none); Supplier 1 Part Number CRA2512-FZ-R010ELFCT-ND -> (none); manf# (none) -> CRA2512-FZ-R010ELF
- U1: #digikey (none) -> 497-7255-1-ND; Manufacturer Part Number L7805CDT-TR -> (none); Supplier 1 Part Number 497-7255-1-ND -> (none); manf# (none) -> L7805CDT-TR
- U2: #digikey (none) -> 296-29100-1-ND; Manufacturer Part Number INA226AIDGST -> (none); Supplier 1 Part Number 296-29100-1-ND -> (none); manf# (none) -> INA226AIDGST
- U3: #digikey (none) -> SN74AHC244QPWRQ1CT-ND; Manufacturer Part Number SN74AHC244QPWRQ1 -> (none); Supplier 1 Part Number SN74AHC244QPWRQ1CT-ND -> (none); manf# (none) -> SN74AHC244QPWRQ1

Commit message: change #digikey to digikey#
Parts:
- C1, C12, C14, C17, C19, C2, C20, C3, C6: #digikey 587-3354-1-ND -> (none); digikey# (none) -> 587-3354-1-ND
- C10, C11, C15, C16: #digikey 490-14410-1-ND -> (none); digikey# (none) -> 490-14410-1-ND
- C13, C18: #digikey 490-14360-1-ND -> (none); digikey# (none) -> 490-14360-1-ND
- C7, C8: #digikey 587-4893-1-ND -> (none); digikey# (none) -> 587-4893-1-ND
- C9: #digikey 1189-1745-ND -> (none); digikey# (none) -> 1189-1745-ND
- D1: #digikey SZMMSZ5240BT1GOSCT-ND -> (none); digikey# (none) -> SZMMSZ5240BT1GOSCT-ND
- D2: #digikey 160-1446-1-ND -> (none); digikey# (none) -> 160-1446-1-ND
- D3: #digikey 160-1448-1-ND -> (none); digikey# (none) -> 160-1448-1-ND
- D4: #digikey 160-1837-1-ND -> (none); digikey# (none) -> 160-1837-1-ND
- FID1, FID2, FID3, FID4, H1, H2, H3, H4, JP1, LOGO1: #digikey dnp -> (none); digikey# (none) -> dnp
- J1: #digikey 277-1128-ND -> (none); digikey# (none) -> 277-1128-ND
- J2: #digikey 609-4277-ND -> (none); digikey# (none) -> 609-4277-ND
- J3: #digikey WM4202-ND -> (none); digikey# (none) -> WM4202-ND
- J4: #digikey WM4305-ND -> (none); digikey# (none) -> WM4305-ND
- JP2: #digikey 732-5316-ND -> (none); digikey# (none) -> 732-5316-ND
- Q1: #digikey IPD90P03P4L04ATMA1CT-ND -> (none); digikey# (none) -> IPD90P03P4L04ATMA1CT-ND
- Q2, Q3: #digikey BTN8982TAAUMA1INCT-ND -> (none); digikey# (none) -> BTN8982TAAUMA1INCT-ND
- R1, R10, R2, R3, R9: #digikey 311-4.7KGRCT-ND -> (none); digikey# (none) -> 311-4.7KGRCT-ND
- R11, R12, R4: #digikey 311-3.3KGRCT-ND -> (none); digikey# (none) -> 311-3.3KGRCT-ND
- R13, R14, R15, R16, R7: #digikey 311-10.0KHRCT-ND -> (none); digikey# (none) -> 311-10.0KHRCT-ND
- R17, R18: #digikey 311-1.00KHRCT-ND -> (none); digikey# (none) -> 311-1.00KHRCT-ND
- R19, R20: #digikey 311-470HRCT-ND -> (none); digikey# (none) -> 311-470HRCT-ND
- R5, R8: #digikey 311-10.0HRCT-ND -> (none); digikey# (none) -> 311-10.0HRCT-ND
- R6: #digikey CRA2512-FZ-R010ELFCT-ND -> (none); digikey# (none) -> CRA2512-FZ-R010ELFCT-ND
- U1: #digikey 497-7255-1-ND -> (none); digikey# (none) -> 497-7255-1-ND
- U2: #digikey 296-29100-1-ND -> (none); digikey# (none) -> 296-29100-1-ND
- U3: #digikey SN74AHC244QPWRQ1CT-ND -> (none); digikey# (none) -> SN74AHC244QPWRQ1CT-ND

Commit message: economic BOM
Parts:
- removed J2: Conn_01x04, Connector_Phoenix_MSTB:PhoenixContact_MSTBVA_2,5_4-G-5,08_1x04_P5.08mm_Vertical, symbol Connector_Generic:Conn_01x04
- added J2, J5: Conn_01x02, Connector_Phoenix_MC_HighVoltage:PhoenixContact_MCV_1,5_2-G-5.08_1x02_P5.08mm_Vertical, symbol Connector_Generic:Conn_01x02
- C1, C12, C14, C17, C19, C2, C20, C3, C6: digikey# 587-3354-1-ND -> 1276-CL10B104KB8WPNDCT-ND; manf# GMK107B7104KAHT -> CL10B104KB8WPND
- C10, C11, C15, C16: digikey# 490-14410-1-ND -> 311-1830-1-ND; manf# GCJ188R71H224KA01D -> CC0603ZRY5V9BB224
- C13, C18: digikey# 490-14360-1-ND -> 399-7842-1-ND; manf# GCM188R91H102KA37D -> C0603C103M5RACTU
- C7, C8: digikey# 587-4893-1-ND -> 490-10505-1-ND; manf# GMK212BBJ106KG-T -> GRM21BC8YA106ME11L
- C9: digikey# 1189-1745-ND -> 1189-3736-1-ND; manf# 35PX1000MEFC10X20 -> 35PK1000MEFCT810X20
- D1: digikey# SZMMSZ5240BT1GOSCT-ND -> BZT52C10-FDICT-ND; manf# SZMMSZ5240BT1G -> BZT52C10-7-F
- D2: value Green led 0603 -> Red led 0603; digikey# 160-1446-1-ND -> 732-4978-1-ND; manf# LTST-C191KGKT -> 150060RS75000
- D3: value Yellow led 0603 -> Red led 0603; digikey# 160-1448-1-ND -> 732-4978-1-ND; manf# LTST-C191KSKT -> 150060RS75000
- D4: value Blue led 0603 -> Red led 0603; digikey# 160-1837-1-ND -> 732-4978-1-ND; manf# LTST-C194TBKT -> 150060RS75000
- J1: footprint Connector_Phoenix_MSTB:PhoenixContact_MSTBVA_2,5_2-G-5,08_1x02_P5.08mm_Vertical -> Connector_Phoenix_MC_HighVoltage:PhoenixContact_MCV_1,5_2-G-5.08_1x02_P5.08mm_Vertical; digikey# 277-1128-ND -> 281-8216-ND; manf# 1758018 -> 1837980000
- Q1: value IPD90P03P4L04 -> IPD50P04P4L11; digikey# IPD90P03P4L04ATMA1CT-ND -> 448-IPD50P04P4L11ATMA2CT-ND; manf# IPD90P03P4L04ATMA1 -> IPD50P04P4L11ATMA2
- Q2, Q3: value BTN8982TA -> BTN8962; digikey# BTN8982TAAUMA1INCT-ND -> BTN8962TAAUMA1; manf# BTN8982TAAUMA1 -> BTN8962TAAUMA1INCT-ND
- U1: digikey# 497-7255-1-ND -> 497-1170-1-ND; manf# L7805CDT-TR -> L7805ABD2T-TR
- U2: digikey# 296-29100-1-ND -> 296-29034-1-ND; manf# INA226AIDGST -> INA226AIDGSR
- U3: digikey# SN74AHC244QPWRQ1CT-ND -> 296-SN74AHC244QPWRQ1CT-ND
Connections:
- net GND: now also J2.1 (Pin_1), J5.2 (Pin_2)
- net at C10.2, C15.1, Q2.4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: now also J2.2 (Pin_2)
- net at C11.2, C16.1, Q3.4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: now also J5.1 (Pin_1)
