File: pcb/dc_motor.kicad_pcb (KiCad board)
At the start: 2 copper layers, 80 x 70 mm, 62 parts, among them J1 Conn_01x02, J2 Conn_01x04, J3 Conn_01x04, J4 Conn_01x07, Q1 IPD90P03P4L04, Q2 BTN8982TA, Q3 BTN8982TA, U1 L7805, U2 INA226, U3 74AHC244

Commit message: routing 01
Parts:
- moved C3 0.63 mm to (103.3, 83.1)
- moved C11 0.20 mm to (92.5, 83.6)
- moved C16 0.20 mm to (91.7, 85.9)
- moved C17 0.20 mm to (94.1, 83.6)
- moved C18 0.20 mm to (90.8, 83.6)
- moved R18 0.20 mm to (89.1, 83.6)
- moved R20 0.20 mm to (85.8, 83.6)
- moved C20 0.20 mm to (87.5, 83.6)
Routing:
- net +5V: track 0.00 -> 77.1 mm, vias 0 -> 12
- net /IS-A: track 0.00 -> 71.1 mm, vias 1 -> 2
- net GND: track 0.00 -> 48.3 mm, vias 18 -> 33
- net /EN_1: track 0.00 -> 48.0 mm
- net /IS-B: track 0.00 -> 39.6 mm
- net VCC: track 0.00 -> 28.4 mm, vias 0 -> 4
- net /PWM2: track 0.00 -> 27.5 mm
- net /PWM1: track 0.00 -> 22.4 mm, vias 0 -> 1
- net Vdrive: track 0.00 -> 20.3 mm
- net Net-(C10-Pad2): track 0.00 -> 19.2 mm, vias 38 -> 36
- net Net-(JP2-Pad2): track 0.00 -> 18.0 mm
- net /EN_2: track 0.00 -> 17.3 mm
- net /A0: track 0.00 -> 16.8 mm
- net /INH-A: track 0.00 -> 16.2 mm, vias 1 -> 0
- net /IN-A: track 0.00 -> 15.2 mm, vias 1 -> 0
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- added copper zone on F.Cu, net GND
- added copper zone on B.Cu, net Net-(C10-Pad2)
- added copper zone on F.Cu, net Net-(C10-Pad2)
- added copper zone on B.Cu, net Net-(C11-Pad2)
- added copper zone on F.Cu, net Net-(C11-Pad2)
- added copper zone on F.Cu, net Net-(C7-Pad1)
- added copper zone on F.Cu, net VCC
- added copper zone on B.Cu, net Vdrive
- added copper zone on F.Cu, net Vdrive
Other:
- board size 80 x 70 mm -> 76 x 70 mm
- net class Default: trace_width 0.25 -> 0.3

Commit message: pcb 01
Parts:
- moved FID3 15.8 mm to (58.0, 100.0)
- moved FID2 5.00 mm to (114.0, 100.0)
- moved FID1 2.00 mm to (114.0, 65.0)
- moved FID4 1.00 mm to (64.0, 58.0)
Routing:
- net GND: track 48.3 -> 63.9 mm, vias 33 -> 139
- net /IS-B: track 39.6 -> 41.4 mm
- net /IS-A: track 71.1 -> 72.3 mm
- net VCC: track 28.4 -> 29.5 mm
- net Vdrive: track 20.3 -> 20.2 mm, vias 18 -> 22
- added copper zone on B.Cu, net GND
Other:
- board text added: "+"
- board text added: "ALE"
- board text added: "EN_1"
- board text added: "GND"
- board text added: "IS_A"
- board text added: "IS_B"
- board text added: "M1+"
- board text added: "M1-"
- board text added: "M2+"
- board text added: "M2-"
- board text added: "PWM1"
- board text added: "PWM2"
- board text added: "SCL"
- board text added: "SDA"
- board text added: "VCC: 8-30v 30A"

Commit message: fix unconnected
Routing:
- net Net-(C11-Pad2): track 14.0 -> 23.2 mm
- net Net-(C10-Pad2): track 18.8 -> 28.0 mm
- net GND: track 63.9 -> 60.4 mm, vias 139 -> 148
Other:
- outline, holes or cut-outs redrawn
- board text added: "01/12/2020"
- board text added: "2 Layers - thickness: 1.6 mm"
- board text added: "Clearance: 0.2 mm"
- board text added: "Grid: 0.1mm"
- board text added: "REV 1.0"
- board text added: "Track Width: 0.3mm"
- board text added: "Via Drill: 0.2mm"
- board text added: "Via size: 0.3mm"
- board text added: "github: Luchao90"
- board text added: "lucianovittori99@gmail.com"
